File: project.kicad_sch (KiCad schematic)
At the start: 0 parts

Commit message: Changed Text Variables and Drawing sheet signature
Other:
- company: ${Department}, ${Company} -> ${Company} ${Department} ${Team}
Changed lines of the file:
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@@
 		(title "${Project}")
 		(rev "${Revision}")
-		(company "${Department}, ${Company}")
+		(company "${Company} ${Department} ${Team}")
 		(comment 1 "${Author}")
 	)
